File: pcb/ECE477_PCB/ECE477_PCB.kicad_pcb (KiCad board)
At the start: 2 copper layers, 65 x 30 mm, 102 parts, among them J1 DEBUG, J10 ToF 5, J11 Pi Zero, J2 USB_B_Micro, J3 ESC, J4 ELRS, J5 AUX_PWR, J6 ToF 1, J7 ToF 2, J8 ToF 3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

Commit message: fixed resistor divider and added keepout under the oscillator
Routing:
- net +3V3: track 206.9 -> 207.8 mm
Changed lines of the file:
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@@
     (property "Sheetname" "")
     (attr smd)
-    (fp_text reference "J3" (at 5.4864 -3.048) (layer "F.SilkS")
+    (fp_text reference "J3" (at 5.4864 -2.3622) (layer "F.SilkS")
       (effects (font (size 0.6 0.6) (thickness 0.15)))
     )
@@
     (property "Sheetname" "")
     (attr smd)
-    (fp_text reference "R25" (at 0 -1.43 90) (layer "F.SilkS")
+    (fp_text reference "R25" (at 0 -1.3208 90) (layer "F.SilkS")
       (effects (font (size 0.6 0.6) (thickness 0.15)))
     )
@@
     (property "Sheetname" "")
     (attr smd)
-    (fp_text reference "R24" (at 0 1.2366 90) (layer "F.SilkS")
+    (fp_text reference "R24" (at 0.0254 -1.3208 90) (layer "F.SilkS")
       (effects (font (size 0.6 0.6) (thickness 0.15)))
     )
@@
     (property "Sheetname" "")
     (attr through_hole)
-    (fp_text reference "J5" (at -1.27 -2.413 90) (layer "F.SilkS")
+    (fp_text reference "J5" (at -0.889 -1.9812 90) (layer "F.SilkS")
       (effects (font (size 0.6 0.6) (thickness 0.15)))
     )
@@
   (via (at 64.5444 36.2854) (size 0.8) (drill 0.4) (layers "F.Cu" "B.Cu") (net 23))
   (via (at 76.1238 37.5666) (size 0.8) (drill 0.4) (layers "F.Cu" "B.Cu") (net 23))
-  (segment (start 64.5444 36.3354) (end 61.0736 39.8062) (width 0.22) (layer "B.Cu") (net 23))
   (segment (start 77.8002 28.6512) (end 79.137 29.988) (width 0.22) (layer "B.Cu") (net 23))
   (segment (start 71.3124 41.0096) (end 72.3302 41.0096) (width 0.22) (layer "B.Cu") (net 23))
@@
   (segment (start 71.8313 31.370536) (end 71.8313 31.192736) (width 0.22) (layer "B.Cu") (net 23))
   (segment (start 68.9102 46.8122) (end 71.82 46.8122) (width 0.22) (layer "B.Cu") (net 23))
+  (segment (start 62.3734 38.5064) (end 61.4426 38.5064) (width 0.22) (layer "B.Cu") (net 23))
   (segment (start 90.0684 50.0126) (end 90.0684 54.102) (width 1.5) (layer "B.Cu") (net 23))
   (segment (start 57.164838 41.189638) (end 57.164838 40.088491) (width 0.22) (layer "B.Cu") (net 23))
@@
   (segment (start 56.3118 47.7012) (end 57.1152 48.5046) (width 0.22) (layer "B.Cu") (net 23))
   (segment (start 77.1652 54.6608) (end 77.9526 54.6608) (width 0.22) (layer "B.Cu") (net 23))
+  (segment (start 61.4426 38.5064) (end 60.6298 39.3192) (width 0.22) (layer "B.Cu") (net 23))
   (segment (start 61.0736 45.0984) (end 57.164838 41.189638) (width 0.22) (layer "B.Cu") (net 23))
   (segment (start 87.249 56.9214) (end 78.8924 56.9214) (width 1.5) (layer "B.Cu") (net 23))
@@
   (segment (start 67.639695 40.3352) (end 67.2894 39.984905) (width 0.22) (layer "B.Cu") (net 23))
   (segment (start 98.1434 47.3184) (end 98.3484 47.5234) (width 1.5) (layer "B.Cu") (net 23))
-  (segment (start 64.5444 36.2854) (end 64.5444 36.3354) (width 0.22) (layer "B.Cu") (net 23))
   (segment (start 65.4326 45.0984) (end 66.6134 45.0984) (width 0.22) (layer "B.Cu") (net 23))
   (segment (start 73.7844 38.9754) (end 75.8476 38.9754) (width 0.22) (layer "B.Cu") (net 23))
@@
   (segment (start 68.2644 41.0096) (end 68.2644 40.959905) (width 0.22) (layer "B.Cu") (net 23))
   (segment (start 95.2754 47.3184) (end 98.1434 47.3184) (width 1.5) (layer "B.Cu") (net 23))
+  (segment (start 60.6298 44.6546) (end 61.0736 45.0984) (width 0.22) (layer "B.Cu") (net 23))
   (segment (start 58.3318 47.7654) (end 58.3692 47.8028) (width 1.5) (layer "B.Cu") (net 23))
+  (segment (start 64.5444 36.3354) (end 62.3734 38.5064) (width 0.22) (layer "B.Cu") (net 23))
   (segment (start 92.7626 47.3184) (end 91.67 48.411) (width 1.5) (layer "B.Cu") (net 23))
   (segment (start 75.8476 38.9754) (end 75.9984 38.8246) (width 0.22) (layer "B.Cu") (net 23))
   (segment (start 76.073 50.48519) (end 76.01408 50.42627) (width 0.22) (layer "B.Cu") (net 23))
+  (segment (start 60.6298 39.3192) (end 60.6298 44.6546) (width 0.22) (layer "B.Cu") (net 23))
   (segment (start 69.737 41.0096) (end 69.0626 40.3352) (width 0.22) (layer "B.Cu") (net 23))
   (segment (start 78.8924 56.9214) (end 58.1152 56.9214) (width 1.5) (layer "B.Cu") (net 23))
   (segment (start 72.3302 41.0096) (end 72.4444 40.8954) (width 0.22) (layer "B.Cu") (net 23))
   (segment (start 77.9526 54.6608) (end 78.6892 55.3974) (width 0.22) (layer "B.Cu") (net 23))
+  (segment (start 64.5444 36.2854) (end 64.5444 36.3354) (width 0.22) (layer "B.Cu") (net 23))
   (segment (start 61.0736 45.0984) (end 66.6134 45.0984) (width 1.5) (layer "B.Cu") (net 23))
   (segment (start 65.3434 45.1876) (end 65.4326 45.0984) (width 0.22) (layer "B.Cu") (net 23))
@@
   (segment (start 57.8544 47.7654) (end 58.3318 47.7654) (width 1.5) (layer "B.Cu") (net 23))
   (segment (start 68.2644 40.959905) (end 67.639695 40.3352) (width 0.22) (layer "B.Cu") (net 23))
-  (segment (start 61.0736 39.8062) (end 61.0736 45.0984) (width 0.22) (layer "B.Cu") (net 23))
   (segment (start 69.7884 41.0096) (end 69.737 41.0096) (width 0.22) (layer "B.Cu") (net 23))
   (segment (start 67.8834 48.7306) (end 67.8834 47.839) (width 0.22) (layer "B.Cu") (net 23))
@@
   (via (at 77.851 48.3616) (size 0.8) (drill 0.4) (layers "F.Cu" "B.Cu") (free) (net 24))
   (via (at 61.4426 47.1424) (size 0.8) (drill 0.4) (layers "F.Cu" "B.Cu") (free) (net 24))
-  (via (at 60.198 43.0784) (size 0.8) (drill 0.4) (layers "F.Cu" "B.Cu") (free) (net 24))
+  (via (at 59.7662 42.2148) (size 0.8) (drill 0.4) (layers "F.Cu" "B.Cu") (free) (net 24))
   (via (at 92.6338 39.497) (size 0.8) (drill 0.4) (layers "F.Cu" "B.Cu") (free) (net 24))
   (via (at 110.3757 42.2976) (size 0.8) (drill 0.4) (layers "F.Cu" "B.Cu") (net 24))
@@
   (via (at 54.9402 51.3334) (size 0.8) (drill 0.4) (layers "F.Cu" "B.Cu") (free) (net 24))
   (via (at 72.263 51.308) (size 0.8) (drill 0.4) (layers "F.Cu" "B.Cu") (free) (net 24))
-  (via (at 59.4106 42.3418) (size 0.8) (drill 0.4) (layers "F.Cu" "B.Cu") (free) (net 24))
+  (via (at 59.7916 41.0718) (size 0.8) (drill 0.4) (layers "F.Cu" "B.Cu") (free) (net 24))
   (via (at 89.2302 35.9664) (size 0.8) (drill 0.4) (layers "F.Cu" "B.Cu") (free) (net 24))
   (via (at 84.3026 39.0398) (size 0.8) (drill 0.4) (layers "F.Cu" "B.Cu") (free) (net 24))
@@
   (via (at 66.3344 48.7354) (size 0.8) (drill 0.4) (layers "F.Cu" "B.Cu") (net 24))
   (via (at 79.0194 38.989) (size 0.8) (drill 0.4) (layers "F.Cu" "B.Cu") (free) (net 24))
-  (via (at 60.2488 41.783) (size 0.8) (drill 0.4) (layers "F.Cu" "B.Cu") (free) (net 24))
+  (via (at 59.6138 39.878) (size 0.8) (drill 0.4) (layers "F.Cu" "B.Cu") (free) (net 24))
   (segment (start 97.2058 55.124298) (end 98.7933 55.124298) (width 0.5) (layer "B.Cu") (net 24))
   (segment (start 110.143899 42.529401) (end 110.3757 42.2976) (width 0.5) (layer "B.Cu") (net 24))
@@
       )
     )
+  )
+  (zone (net 0) (net_name "") (layer "B.Cu") (hatch edge 0.508)
+    (connect_pads (clearance 0))
+    (min_thickness 0.254)
+    (keepout (tracks not_allowed) (vias not_allowed) (pads not_allowed) (copperpour not_allowed) (footprints not_allowed))
+    (fill (thermal_gap 0.508) (thermal_bridge_width 0.508))
+    (polygon
+      (pts
+        (xy 64.5922 44.2214)
+        (xy 61.2902 44.2214)
+        (xy 61.2902 39.0144)
+        (xy 64.5922 39.0144)
+      )
+    )

Commit message: extended qfn pads, added 3d model
Parts:
- moved R27 0.58 mm to (60.0, 53.8)
- moved C26 0.46 mm to (62.7, 51.0)
- moved R26 0.32 mm to (77.9, 49.3)
Routing:
- net Net-(R22-Pad2): track 25.4 -> 26.8 mm
- net SPI1_SCK: track 23.5 -> 24.6 mm
- net Net-(R27-Pad1): track 13.0 -> 14.0 mm
- net +3V3: track 207.8 -> 208.8 mm
- net GND: track 20.5 -> 21.1 mm
