File: pcb/ECE477_PCB/ECE477_PCB.kicad_sch (KiCad schematic)
At the start: 91 parts, among them J1 DEBUG, J10 ToF 5, J11 Pi Zero, J2 USB_B_Micro, J3 ESC, J4 ELRS, J5 AUX_PWR, J6 ToF 1, J7 ToF 2, J8 ToF 3, J9 ToF 4, M1 Brushed_DC, M2 Brushed_DC, M3 Brushed_DC, M4 Brushed_DC, Q1 IRLML6244TR, Q2 IRLML6244TR, Q3 IRLML6244TR, Q4 IRLML6244TR, SW1 RESET, U1 STM32F446RETx, U2 Pololu_S13V10F5, U3 REG1117-3.3, U4 FT230XQ, Y1 16MHz X322516MLB4SI

Commit message: last fixes, ready to order (I think)
Parts:
- added C28: 1uF, Capacitor_SMD:C_0603_1608Metric, symbol Device:C_Small
Connections:
- net GND: now also C28.1
- net VSENSE: now also C28.2
Changed lines of the file:
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@@
   (junction (at 54.61 143.51) (diameter 0) (color 0 0 0 0)
   )
+  (junction (at 130.81 145.415) (diameter 0) (color 0 0 0 0)
+  )
+  (junction (at 146.685 135.89) (diameter 0) (color 0 0 0 0)
+  )
   (junction (at 66.04 55.88) (diameter 0) (color 0 0 0 0)
   )
@@
     (stroke (width 0) (type default) (color 0 0 0 0))
   )
+  (wire (pts (xy 130.81 145.415) (xy 130.81 146.05))
+    (stroke (width 0) (type default) (color 0 0 0 0))
+  )
   (wire (pts (xy 177.8 104.14) (xy 177.8 100.33))
     (stroke (width 0) (type default) (color 0 0 0 0))
@@
     (stroke (width 0) (type default) (color 0 0 0 0))
   )
+  (wire (pts (xy 146.685 143.51) (xy 146.685 145.415))
+    (stroke (width 0) (type default) (color 0 0 0 0))
+  )
   (wire (pts (xy 137.16 101.6) (xy 140.97 101.6))
     (stroke (width 0) (type default) (color 0 0 0 0))
@@
     (stroke (width 0) (type default) (color 0 0 0 0))
   )
-  (wire (pts (xy 130.81 144.78) (xy 130.81 146.05))
+  (wire (pts (xy 130.81 144.78) (xy 130.81 145.415))
     (stroke (width 0) (type default) (color 0 0 0 0))
   )
@@
     (stroke (width 0) (type default) (color 0 0 0 0))
   )
+  (wire (pts (xy 146.685 135.89) (xy 150.495 135.89))
+    (stroke (width 0) (type default) (color 0 0 0 0))
+  )
   (wire (pts (xy 226.06 74.93) (xy 228.6 74.93))
     (stroke (width 0) (type default) (color 0 0 0 0))
@@
     (stroke (width 0) (type default) (color 0 0 0 0))
   )
+  (wire (pts (xy 146.685 135.89) (xy 146.685 138.43))
+    (stroke (width 0) (type default) (color 0 0 0 0))
+  )
   (wire (pts (xy 149.86 85.09) (xy 149.86 86.36))
     (stroke (width 0) (type default) (color 0 0 0 0))
@@
     (stroke (width 0) (type default) (color 0 0 0 0))
   )
+  (wire (pts (xy 146.685 145.415) (xy 130.81 145.415))
+    (stroke (width 0) (type default) (color 0 0 0 0))
+  )
   (wire (pts (xy 194.31 33.02) (xy 193.04 33.02))
     (stroke (width 0) (type default) (color 0 0 0 0))
@@
     (stroke (width 0) (type default) (color 0 0 0 0))
   )
-  (wire (pts (xy 143.51 135.89) (xy 144.78 135.89))
+  (wire (pts (xy 143.51 135.89) (xy 146.685 135.89))
     (stroke (width 0) (type default) (color 0 0 0 0))
   )
@@
     )
   )
-  (global_label "VSENSE" (shape input) (at 144.78 135.89 0) (fields_autoplaced)
+  (global_label "VSENSE" (shape input) (at 150.495 135.89 0) (fields_autoplaced)
     (effects (font (size 1.27 1.27)) (justify left))
-    (property "Intersheet References" "${INTERSHEET_REFS}" (id 0) (at -11.43 12.7 0)
+    (property "Intersheet References" "${INTERSHEET_REFS}" (id 0) (at -5.715 12.7 0)
       (effects (font (size 1.27 1.27)) hide)
     )
@@
     (pin "1")
   )
+  (symbol (lib_id "Device:C_Small") (at 146.685 140.97 180) (unit 1)
+    (in_bom yes) (on_board yes)
+    (property "Reference" "C28" (id 0) (at 144.145 142.24 0)
+      (effects (font (size 1.27 1.27)) (justify left))
+    )
+    (property "Value" "1uF" (id 1) (at 144.145 139.7 0)
+      (effects (font (size 1.27 1.27)) (justify left))
+    )
+    (property "Footprint" "Capacitor_SMD:C_0603_1608Metric" (id 2) (at 146.685 140.97 0)
+      (effects (font (size 1.27 1.27)) hide)
+    )
+    (property "Datasheet" "~" (id 3) (at 146.685 140.97 0)
+      (effects (font (size 1.27 1.27)) hide)
+    )
+    (property "LCSC Part #" "C15849" (id 4) (at 146.685 140.97 0)
+      (effects (font (size 1.27 1.27)) hide)
+    )
+    (property "LCSC" "C15849" (id 5) (at 146.685 140.97 0)
+      (effects (font (size 1.27 1.27)) hide)
+    )
+    (pin "1")
+    (pin "2")
+  )
   (symbol (lib_id "power:GND") (at 153.67 106.68 0) (unit 1)
     (in_bom yes) (on_board yes)
@@
       (reference "C27") (unit 1) (value "0.1uF 4V") (footprint "Capacitor_SMD:C_0603_1608Metric")
     )
+    (path "/a8794c00-0369-4d64-970e-4d522e322130"
+      (reference "C28") (unit 1) (value "1uF") (footprint "Capacitor_SMD:C_0603_1608Metric")
+    )
     (path "/0312643c-df93-4304-9858-72b871182e4e"
